File: PQDB-HW-Kicad/Base.sch (KiCad schematic (older format))
At the start: 70 parts, among them Q101 BC847, Q102 BC847, Q201 BC847, Q301 BC847, Q302 BC847, Q303 BC847, Q304 BC847, SW101 BTN-01, SW102 BTN-01, SW103 BTN-01, SW104 BTN-01, SW105 BTN-01, SW106 BTN-01, SW107 BTN-01, SW108 BTN-01, SW109 BTN-01, SW110 BTN-01, U201 LM35, U301 KW4-361, U401 DISPLAY_JHD162A, U601 74HC595, U701 DS1307Z, X701 32.768 KHz

Commit message: Add files via upload
Parts:
- removed RV201, RV401: POT, HW_Footprints:HW_Potenciometro_2, symbol POT
- added P101: EXT_I2C, bibliotecas:EXT_I2C, symbol EXT_I2C
- added R105, R106: 1k, bibliotecas:HW_Resistor, symbol RSMALL
- added RV201, RV401: POT_DUPLO, bibliotecas:HW_Potenciometro_2_Duplo, symbol POT_DUPLO
- BT701: footprint HW_Footprints:HW_CR2032H -> bibliotecas:HW_CR2032H
- BZ201: footprint HW_Footprints:HW_Buzzer -> bibliotecas:HW_Buzzer
- C701: footprint HW_Footprints:HW_CAPACITOR -> bibliotecas:HW_CAPACITOR
- R101, R102, R103, R104, R201, R202, R301, R302, R303, R304, R305, R306, R307, R308, R309, R310, R311, R312, R401, R406, R407, R408, R501, R502, R503, R701, R702: footprint HW_Footprints:HW_Resistor -> bibliotecas:HW_Resistor
- R601, R602: footprint Resistors_ThroughHole:Resistor_Horizontal_RM15mm -> bibliotecas:Resistor_Horizontal_RM15mm
- RGB501: footprint HW_Footprints:HW_LED-5MM-RGB -> bibliotecas:LED-5MM
- SHIELD801: footprint arduino_shields:ARDUINO_SHIELD_2 -> bibliotecas:ARDUINO_SHIELD_2
- SW101, SW102, SW103, SW104, SW105, SW106, SW107, SW108, SW109, SW110: footprint HW_Footprints:HW_Switch_tactil_adaptada -> bibliotecas:HW_Switch_tactil_adaptada
- U201: footprint HW_Footprints:HW_TO92-123 -> bibliotecas:TO-92_Molded_Narrow_Reverse
- U301: footprint HW_Footprints:HW_Disp_7seg_4dig -> bibliotecas:HW_Disp_7seg_4dig
- U401: footprint HW_Footprints:HW_LCD -> bibliotecas:HW_LCD
- U601: footprint HW_Footprints:HW_DIP-16__300_ELL -> bibliotecas:HW_DIP-16__300_ELL
- U701: footprint HW_Footprints:HW_DIP-8 -> bibliotecas:DIP-8_W7.62mm_LongPads
- X701: footprint HW_Footprints:HW_Crystal_32768 -> bibliotecas:Crystal_Round_Horizontal_2mm
Connections:
- net +5V: now also P101.1 (5V), RV401.3
- net 3V3: now also RV201.3
- net AN2: now also RV201.2
- net GND: now also P101.2 (GND), R105.2, R106.1, RV201.1, RV401.1
- net SCL: now also P101.4 (SCL)
- net SDA: now also P101.3 (SDA)
- net VEE: now also RV401.2
- net at R103.2, SW101.1, SW103.1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: now also R105.1
- net at R104.2, SW102.1, SW104.1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: now also R106.2
Other:
- note added: "Extensão I2C"
- moved on the sheet: BT701, BZ201, D101, D102, D103, D104, D105, D106, D107, D108, D109, D110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
