File: PQDB-Mini-HW-Kicad/Base.kicad_pcb (KiCad board)
At the start: 2 copper layers, 99.6 x 50 mm, 72 parts, among them Q101 BC847, Q102 BC847, Q201 BC847, Q301 BC847, Q302 BC847, Q303 BC847, Q304 BC847, SW101 BTN-01, SW102 BTN-01, SW103 BTN-01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

Commit message: Add files via upload
Parts:
- added G***: LOGO, bibliotecas:OSHW_PEQ, F.Cu at (116.3, 107.2)
- added G***: LOGO, bibliotecas:UNIFEI_PEQ, F.Cu at (174.6, 107.3)
- added P101: EXT_I2C, bibliotecas:EXT_I2C, F.Cu at (110.2, 68.5)
- added REF**: 1pin, Connectors:1pin, F.Cu at (125.3, 65.8)
- added REF**: 1pin, Connectors:1pin, F.Cu at (165.5, 65.8)
- D101, D102, D103, D104, D105, D106, D107, D108, D109, D110: footprint Resistors_SMD:R_0805_HandSoldering -> bibliotecas:R_0805_HandSoldering
- RV201, RV202: value POT -> POT_DUPLO; footprint bibliotecas:HW_Potenciometro_2 -> bibliotecas:HW_Potenciometro_2_Duplo
- SW101, SW102, SW103, SW104, SW105, SW106, SW107, SW108, SW109, SW110: footprint Buttons_Switches_ThroughHole:SW_PUSH_6mm -> bibliotecas:SW_PUSH_6mm
- moved D108 93.6 mm to (192.4, 95.0), turned to 315 degrees
- moved D105 87.0 mm to (105.5, 101.8), turned to 225 degrees
- moved SW108 84.2 mm to (190.0, 102.5), turned to 135 degrees
- moved D107 80.6 mm to (98.7, 95.3), turned to 225 degrees
- moved D106 80.3 mm to (185.7, 101.8), turned to 315 degrees
- moved D109 80.0 mm to (105.6, 88.5), turned to 225 degrees
- moved D110 80.0 mm to (185.7, 88.8), turned to 315 degrees
- moved SW105 77.7 mm to (112.3, 104.0), turned to 225 degrees
- moved D103 74.3 mm to (111.9, 95.1), turned to 225 degrees
- moved SW106 71.4 mm to (183.5, 108.7), turned to 135 degrees
- moved SW107 71.2 mm to (106.0, 97.7), turned to 225 degrees
- moved SW109 70.9 mm to (112.6, 91.2), turned to 225 degrees
- moved SW110 70.9 mm to (183.3, 95.8), turned to 135 degrees
- moved D104 67.2 mm to (179.2, 95.1), turned to 315 degrees
- moved SW103 65.8 mm to (118.8, 97.6), turned to 225 degrees
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Connections:
- Q101 pad 2: /T1 -> /T2
- Q102 pad 2: /T2 -> /T1
- R101 pad 1: /T1 -> /T2
- R102 pad 1: /T2 -> /T1
- SW101 pad 1: Net-(R103-Pad2) -> Net-(R104-Pad2)
- SW102 pad 1: Net-(R104-Pad2) -> Net-(R103-Pad2)
- SW103 pad 1: Net-(R103-Pad2) -> Net-(R104-Pad2)
- SW104 pad 1: Net-(R104-Pad2) -> Net-(R103-Pad2)
- SW105 pad 1: Net-(R103-Pad2) -> Net-(R104-Pad2)
- SW106 pad 1: Net-(R104-Pad2) -> Net-(R103-Pad2)
- SW107 pad 1: Net-(R103-Pad2) -> Net-(R104-Pad2)
- SW108 pad 1: Net-(R104-Pad2) -> Net-(R103-Pad2)
- SW109 pad 1: Net-(R103-Pad2) -> Net-(R104-Pad2)
- SW110 pad 1: Net-(R104-Pad2) -> Net-(R103-Pad2)
Routing:
- net GND: track 175.2 -> 216.0 mm
- net /T1: track 44.8 -> 85.4 mm
- net /T2: track 76.6 -> 36.8 mm, vias 3 -> 2
- net /SDA: track 32.9 -> 71.3 mm, vias 2 -> 4
- net +5V: track 145.4 -> 175.1 mm, vias 6 -> 8
- net /SCL: track 43.3 -> 71.8 mm, vias 1 -> 3
- net /D4: track 109.3 -> 127.0 mm, vias 6 -> 10
- net /D6: track 93.2 -> 81.8 mm, vias 4 -> 2
- net Net-(U701-Pad1): track 2.52 -> 10.0 mm
- net Net-(U701-Pad2): track 4.84 -> 11.6 mm
- net /D5: track 130.8 -> 125.4 mm, vias 8 -> 4
- net Net-(R406-Pad2): track 10.5 -> 7.19 mm
- net Net-(R703-Pad2): track 7.57 -> 6.09 mm
- net Net-(D108-Pad2): track 9.37 -> 10.6 mm
- net Net-(R402-Pad2): track 44.0 -> 45.2 mm, vias 1 -> 2
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Other:
- board size 99.6 x 50 mm -> 99.6 x 50.4 mm
- board text added: "5V GND SDA SCL"
- board text added: "Licensed under CERN OHL v.1.2"
- board text added: "RV201"
- board text added: "RV202"
- board text removed: "ALFA RMAA"
