File: PQDB-Mini-HW-Kicad/Base.sch (KiCad schematic (older format))
At the start: 72 parts, among them Q101 BC847, Q102 BC847, Q201 BC847, Q301 BC847, Q302 BC847, Q303 BC847, Q304 BC847, SW101 BTN-01, SW102 BTN-01, SW103 BTN-01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

Commit message: Add files via upload
Parts:
- removed RV201, RV202: POT, bibliotecas:HW_Potenciometro_2, symbol POT-RESCUE-Base
- added P101: EXT_I2C, bibliotecas:EXT_I2C, symbol EXT_I2C
- added RV201, RV202: POT_DUPLO, bibliotecas:HW_Potenciometro_2_Duplo, symbol POT_DUPLO
- D101: renamed from D102; footprint Diodes_SMD:MiniMELF_Handsoldering -> bibliotecas:R_0805_HandSoldering
- D102: renamed from D101; footprint Diodes_SMD:MiniMELF_Handsoldering -> bibliotecas:R_0805_HandSoldering
- D103: renamed from D104; footprint Diodes_SMD:MiniMELF_Handsoldering -> bibliotecas:R_0805_HandSoldering
- D104: renamed from D103; footprint Diodes_SMD:MiniMELF_Handsoldering -> bibliotecas:R_0805_HandSoldering
- D105: renamed from D106; footprint Diodes_SMD:MiniMELF_Handsoldering -> bibliotecas:R_0805_HandSoldering
- D106: renamed from D105; footprint Diodes_SMD:MiniMELF_Handsoldering -> bibliotecas:R_0805_HandSoldering
- D107: renamed from D108; footprint Diodes_SMD:MiniMELF_Handsoldering -> bibliotecas:R_0805_HandSoldering
- D108: renamed from D107; footprint Diodes_SMD:MiniMELF_Handsoldering -> bibliotecas:R_0805_HandSoldering
- D109: renamed from D110; footprint Diodes_SMD:MiniMELF_Handsoldering -> bibliotecas:R_0805_HandSoldering
- D110: renamed from D109; footprint Diodes_SMD:MiniMELF_Handsoldering -> bibliotecas:R_0805_HandSoldering
- SW101: renamed from SW102; footprint bibliotecas:HW_Switch_tactil_adaptada -> bibliotecas:SW_PUSH_6mm
- SW102: renamed from SW101; footprint bibliotecas:HW_Switch_tactil_adaptada -> bibliotecas:SW_PUSH_6mm
- SW103: renamed from SW104; footprint bibliotecas:HW_Switch_tactil_adaptada -> bibliotecas:SW_PUSH_6mm
- SW104: renamed from SW103; footprint bibliotecas:HW_Switch_tactil_adaptada -> bibliotecas:SW_PUSH_6mm
- SW105: renamed from SW106; footprint bibliotecas:HW_Switch_tactil_adaptada -> bibliotecas:SW_PUSH_6mm
- SW106: renamed from SW105; footprint bibliotecas:HW_Switch_tactil_adaptada -> bibliotecas:SW_PUSH_6mm
- SW107: renamed from SW108; footprint bibliotecas:HW_Switch_tactil_adaptada -> bibliotecas:SW_PUSH_6mm
- SW108: renamed from SW107; footprint bibliotecas:HW_Switch_tactil_adaptada -> bibliotecas:SW_PUSH_6mm
- SW109: renamed from SW110; footprint bibliotecas:HW_Switch_tactil_adaptada -> bibliotecas:SW_PUSH_6mm
- SW110: renamed from SW109; footprint bibliotecas:HW_Switch_tactil_adaptada -> bibliotecas:SW_PUSH_6mm
Connections:
- net +5V: now also P101.1 (5V)
- net 3V3: now also RV201.3, RV202.3
- net AN2: now also RV201.2
- net AN3: now also RV202.2
- net GND: now also P101.2 (GND), RV201.1, RV202.1
- net SCL: now also P101.4 (SCL)
- net SDA: now also P101.3 (SDA)
- net T1: now also Q102.2 (E), R102.1; no longer Q101.2 (E), R101.1
- net T2: now also Q101.2 (E), R101.1; no longer Q102.2 (E), R102.1
Other:
- note added: "Display Nokia 5110"
- note added: "Extensão I2C"
- moved on the sheet: R401, R402, R403, R404, R405, R406, U401
